Commit message: improved sim launch files and updated usage instructions

File: my_robot/description/urdf/romi.urdf.xacro (robot description, xacro)
@@ -1,13 +1,16 @@
 <?xml version="1.0"?>
 <robot xmlns:xacro="http://www.ros.org/wiki/xacro" name="robot">
+    <!-- Accept argument to enable/disable simulation-specific configuration -->
+    <xacro:arg name="use_simulation" default="false"/>
     <xacro:include filename="romi_core.xacro"/>
     <!-- <xacro:include filename="romi_camera.xacro"/> -->
     <xacro:include filename="romi_lidar.xacro"/>
     <!-- For sim only -->
-    <!-- <gazebo>
-        <plugin name="gazebo_ros_control" filename="libgazebo_ros_control.so">
-        <robotNamespace>robot</robotNamespace>
-        </plugin>
-    </gazebo> -->
+    <xacro:if value="$(arg use_simulation)">
+        <gazebo>
+            <plugin name="gazebo_ros_control" filename="libgazebo_ros_control.so">
+            </plugin>
+        </gazebo>
+    </xacro:if>
     <transmission name="left_wheel_transmission">
         <type>transmission_interface/SimpleTransmission</type>

File: my_robot/description/urdf/romi_lidar.xacro (robot description, xacro)
@@ -13,9 +13,4 @@
             <material name="black"/>
         </visual>
-        <collision>
-            <geometry>
-                <cylinder radius="0.05" length="0.04"/>
-            </geometry>
-        </collision>
     </link>
     <gazebo reference="lidar_frame">
